File: kicad/B1024.kicad_pcb (KiCad board)
At the start: 2 copper layers, 1 part

Commit message: Add remaining parts, prelim board layout
Rotated pictures to match board layout. Added missing ics, resistors,
and jumpers. Preliminary layout. Updated readme.
Parts:
- removed REF**: DIP-16_W7.62mm, Package_DIP:DIP-16_W7.62mm
- added C1: 0.1uf, Capacitor_THT:C_Disc_D4.7mm_W2.5mm_P5.00mm, F.Cu at (94.9, 22.1)
- added C10: 0.1uf, Capacitor_THT:C_Disc_D4.7mm_W2.5mm_P5.00mm, F.Cu at (91.7, 148.4)
- added C11: 0.1uf, Capacitor_THT:C_Disc_D4.7mm_W2.5mm_P5.00mm, F.Cu at (131.3, 23.3)
- added C12: 0.1uf, Capacitor_THT:C_Disc_D4.7mm_W2.5mm_P5.00mm, F.Cu at (143.0, 23.3)
- added C13: 0.1uf, Capacitor_THT:C_Disc_D4.7mm_W2.5mm_P5.00mm, F.Cu at (154.5, 23.3)
- added C14: 0.1uf, Capacitor_THT:C_Disc_D4.7mm_W2.5mm_P5.00mm, F.Cu at (167.1, 23.3)
- added C15: 0.1uf, Capacitor_THT:C_Disc_D4.7mm_W2.5mm_P5.00mm, F.Cu at (178.6, 23.3)
- added C16: 0.1uf, Capacitor_THT:C_Disc_D4.7mm_W2.5mm_P5.00mm, F.Cu at (191.1, 23.3)
- added C17: 0.1uf, Capacitor_THT:C_Disc_D4.7mm_W2.5mm_P5.00mm, F.Cu at (202.2, 23.3)
- added C18: 0.1uf, Capacitor_THT:C_Disc_D4.7mm_W2.5mm_P5.00mm, F.Cu at (214.4, 23.3)
- added C19: 0.1uf, Capacitor_THT:C_Disc_D4.7mm_W2.5mm_P5.00mm, F.Cu at (131.3, 56.0)
- added C2: 0.1uf, Capacitor_THT:C_Disc_D4.7mm_W2.5mm_P5.00mm, F.Cu at (95.1, 43.0)
- added C20: 0.1uf, Capacitor_THT:C_Disc_D4.7mm_W2.5mm_P5.00mm, F.Cu at (142.7, 55.8)
- added C21: 0.1uf, Capacitor_THT:C_Disc_D4.7mm_W2.5mm_P5.00mm, F.Cu at (154.6, 55.6)
- added C22: 0.1uf, Capacitor_THT:C_Disc_D4.7mm_W2.5mm_P5.00mm, F.Cu at (166.2, 55.7)
- added C23: 0.1uf, Capacitor_THT:C_Disc_D4.7mm_W2.5mm_P5.00mm, F.Cu at (178.5, 55.9)
- added C24: 0.1uf, Capacitor_THT:C_Disc_D4.7mm_W2.5mm_P5.00mm, F.Cu at (202.1, 56.1)
- added C25: 0.1uf, Capacitor_THT:C_Disc_D4.7mm_W2.5mm_P5.00mm, F.Cu at (214.5, 56.1)
- added C26: 0.1uf, Capacitor_THT:C_Disc_D4.7mm_W2.5mm_P5.00mm, F.Cu at (131.3, 88.2)
- added C27: 0.1uf, Capacitor_THT:C_Disc_D4.7mm_W2.5mm_P5.00mm, F.Cu at (143.3, 88.3)
- added C28: 0.1uf, Capacitor_THT:C_Disc_D4.7mm_W2.5mm_P5.00mm, F.Cu at (154.9, 88.2)
- added C29: 0.1uf, Capacitor_THT:C_Disc_D4.7mm_W2.5mm_P5.00mm, F.Cu at (166.4, 88.0)
- added C3: 0.1uf, Capacitor_THT:C_Disc_D4.7mm_W2.5mm_P5.00mm, F.Cu at (95.1, 54.7)
- added C30: 0.1uf, Capacitor_THT:C_Disc_D4.7mm_W2.5mm_P5.00mm, F.Cu at (190.6, 56.0)
- added C31: 0.1uf, Capacitor_THT:C_Disc_D4.7mm_W2.5mm_P5.00mm, F.Cu at (178.6, 88.0)
- added C32: 0.1uf, Capacitor_THT:C_Disc_D4.7mm_W2.5mm_P5.00mm, F.Cu at (190.5, 88.2)
- added C33: 0.1uf, Capacitor_THT:C_Disc_D4.7mm_W2.5mm_P5.00mm, F.Cu at (202.4, 88.0)
- added C34: 0.1uf, Capacitor_THT:C_Disc_D4.7mm_W2.5mm_P5.00mm, F.Cu at (214.3, 88.0)
- added C35: 0.1uf, Capacitor_THT:C_Disc_D4.7mm_W2.5mm_P5.00mm, F.Cu at (131.5, 119.6)
- added C36: 0.1uf, Capacitor_THT:C_Disc_D4.7mm_W2.5mm_P5.00mm, F.Cu at (143.1, 119.5)
- added C37: 0.1uf, Capacitor_THT:C_Disc_D4.7mm_W2.5mm_P5.00mm, F.Cu at (155.0, 119.7)
- added C38: 0.1uf, Capacitor_THT:C_Disc_D4.7mm_W2.5mm_P5.00mm, F.Cu at (166.8, 119.3)
- added C39: 0.1uf, Capacitor_THT:C_Disc_D4.7mm_W2.5mm_P5.00mm, F.Cu at (178.9, 119.4)
- added C4: 0.1uf, Capacitor_THT:C_Disc_D4.7mm_W2.5mm_P5.00mm, F.Cu at (102.2, 64.9)
- added C40: 0.1uf, Capacitor_THT:C_Disc_D4.7mm_W2.5mm_P5.00mm, F.Cu at (190.9, 119.1)
- added C41: 0.1uf, Capacitor_THT:C_Disc_D4.7mm_W2.5mm_P5.00mm, F.Cu at (202.7, 119.5)
- added C42: 0.1uf, Capacitor_THT:C_Disc_D4.7mm_W2.5mm_P5.00mm, F.Cu at (214.2, 119.2)
- added C43: 0.1uf, Capacitor_THT:C_Disc_D4.7mm_W2.5mm_P5.00mm, F.Cu at (131.2, 149.3)
- added C44: 0.1uf, Capacitor_THT:C_Disc_D4.7mm_W2.5mm_P5.00mm, F.Cu at (143.4, 149.5)
- added C45: 0.1uf, Capacitor_THT:C_Disc_D4.7mm_W2.5mm_P5.00mm, F.Cu at (155.7, 149.5)
- added C46: 0.1uf, Capacitor_THT:C_Disc_D4.7mm_W2.5mm_P5.00mm, F.Cu at (166.8, 149.4)
- added C47: 0.1uf, Capacitor_THT:C_Disc_D4.7mm_W2.5mm_P5.00mm, F.Cu at (179.5, 149.3)
- added C48: 0.1uf, Capacitor_THT:C_Disc_D4.7mm_W2.5mm_P5.00mm, F.Cu at (191.2, 149.9)
- added C49: 0.1uf, Capacitor_THT:C_Disc_D4.7mm_W2.5mm_P5.00mm, F.Cu at (203.0, 150.3)
- added C5: 0.1uf, Capacitor_THT:C_Disc_D4.7mm_W2.5mm_P5.00mm, F.Cu at (91.4, 81.6)
- added C50: 0.1uf, Capacitor_THT:C_Disc_D4.7mm_W2.5mm_P5.00mm, F.Cu at (215.1, 150.1)
- added C51: 0.1uf, Capacitor_THT:C_Disc_D4.7mm_W2.5mm_P5.00mm, F.Cu at (236.5, 33.7)
- added C52: 0.1uf, Capacitor_THT:C_Disc_D4.7mm_W2.5mm_P5.00mm, F.Cu at (237.9, 57.2)
- added C6: 0.1uf, Capacitor_THT:C_Disc_D4.7mm_W2.5mm_P5.00mm, F.Cu at (91.2, 95.3)
- added C7: 0.1uf, Capacitor_THT:C_Disc_D4.7mm_W2.5mm_P5.00mm, F.Cu at (91.3, 108.7)
- added C8: 0.1uf, Capacitor_THT:C_Disc_D4.7mm_W2.5mm_P5.00mm, F.Cu at (91.4, 121.8)
- added C9: 0.1uf, Capacitor_THT:C_Disc_D4.7mm_W2.5mm_P5.00mm, F.Cu at (91.6, 135.4)
- added J1: "RESET", Connector_PinHeader_2.54mm:PinHeader_1x02_P2.54mm_Horizontal, F.Cu at (47.4, 45.5)
- added J2: "0FFF/0800 EN", Connector_PinHeader_2.54mm:PinHeader_1x03_P2.54mm_Horizontal, F.Cu at (83.3, 63.8)
- added J3: "LED", Connector_PinHeader_2.54mm:PinHeader_1x03_P2.54mm_Horizontal, F.Cu at (44.7, 142.5)
- added J4: "RAM ROM", Connector_PinHeader_2.54mm:PinHeader_1x03_P2.54mm_Horizontal, F.Cu at (50.3, 148.7)
- added J5: EXP, Connector_PinHeader_2.54mm:PinHeader_2x30_P2.54mm_Vertical, F.Cu at (74.3, 52.6)
- added J6: EXP, Connector_PinHeader_2.54mm:PinHeader_2x30_P2.54mm_Vertical, F.Cu at (60.7, 52.7)
- added J9: COPRO, Connector_PinHeader_2.54mm:PinHeader_2x20_P2.54mm_Vertical, F.Cu at (264.3, 81.4)
- added P7: EXP, Connector_PinHeader_2.54mm:PinHeader_2x30_P2.54mm_Vertical, F.Cu at (38.9, 52.5)
- added P9: COPRO, Connector_PinHeader_2.54mm:PinHeader_2x20_P2.54mm_Vertical, F.Cu at (228.0, 81.4)
- added R1: 22ohm, Resistor_THT:R_Axial_DIN0207_L6.3mm_D2.5mm_P10.16mm_Horizontal, F.Cu at (44.8, 133.4)
- added R2: 4K7, Resistor_THT:R_Axial_DIN0207_L6.3mm_D2.5mm_P10.16mm_Horizontal, F.Cu at (122.3, 37.1)
- added R3: 4K7, Resistor_THT:R_Axial_DIN0207_L6.3mm_D2.5mm_P10.16mm_Horizontal, F.Cu at (122.3, 62.5)
- added R4: 22ohm, Resistor_THT:R_Axial_DIN0207_L6.3mm_D2.5mm_P10.16mm_Horizontal, F.Cu at (227.5, 152.8)
- added RN1: 4K7, Resistor_THT:R_Array_SIP10, F.Cu at (55.4, 137.5)
- added RN2: 22 ohm, Resistor_THT:R_Array_SIP10, F.Cu at (123.7, 89.0)
- added RN3: 22 ohm, Resistor_THT:R_Array_SIP10, F.Cu at (123.7, 139.9)
- added RN4: 22 ohm, Resistor_THT:R_Array_SIP8, F.Cu at (227.5, 21.0)
- added RN5: 22 ohm, Resistor_THT:R_Array_SIP8, F.Cu at (227.9, 46.5)
- added RN6: 4K7, Resistor_THT:R_Array_SIP8, F.Cu at (234.3, 50.5)
- added RN7: 10K, Resistor_THT:R_Array_SIP10, F.Cu at (248.7, 78.5)
- added RN8: 10K, Resistor_THT:R_Array_SIP10, F.Cu at (253.5, 78.6)
- added RN9: 4K7, Resistor_THT:R_Array_SIP8, F.Cu at (233.6, 136.8)
- added U1: 6264, Package_DIP:DIP-28_W15.24mm, F.Cu at (45.6, 37.4)
- added U10: 74153, Package_DIP:DIP-16_W7.62mm, F.Cu at (96.3, 136.4)
- added U11: 74153, Package_DIP:DIP-16_W7.62mm, F.Cu at (96.3, 149.8)
- added U12: 41256, Package_DIP:DIP-16_W7.62mm, F.Cu at (129.8, 29.9)
- added U13: 41256, Package_DIP:DIP-16_W7.62mm, F.Cu at (141.8, 29.8)
- added U14: 41256, Package_DIP:DIP-16_W7.62mm, F.Cu at (153.7, 29.8)
- added U15: 41256, Package_DIP:DIP-16_W7.62mm, F.Cu at (165.6, 29.8)
- added U16: 41256, Package_DIP:DIP-16_W7.62mm, F.Cu at (177.5, 29.8)
- added U17: 41256, Package_DIP:DIP-16_W7.62mm, F.Cu at (189.4, 29.8)
- added U18: 41256, Package_DIP:DIP-16_W7.62mm, F.Cu at (201.4, 29.8)
- added U19: 41256, Package_DIP:DIP-16_W7.62mm, F.Cu at (213.3, 29.8)
- added U2: 74LS85, Package_DIP:DIP-16_W7.62mm, F.Cu at (58.7, 149.0)
- added U20: 41256, Package_DIP:DIP-16_W7.62mm, F.Cu at (129.5, 63.2)
- added U21: 41256, Package_DIP:DIP-16_W7.62mm, F.Cu at (141.4, 63.1)
- added U22: 41256, Package_DIP:DIP-16_W7.62mm, F.Cu at (153.3, 63.1)
- added U23: 41256, Package_DIP:DIP-16_W7.62mm, F.Cu at (165.2, 63.1)
- added U24: 41256, Package_DIP:DIP-16_W7.62mm, F.Cu at (177.2, 63.1)
- added U25: 41256, Package_DIP:DIP-16_W7.62mm, F.Cu at (189.1, 63.1)
- added U26: 41256, Package_DIP:DIP-16_W7.62mm, F.Cu at (201.0, 63.1)
- added U27: 41256, Package_DIP:DIP-16_W7.62mm, F.Cu at (212.9, 63.1)
- added U28: 41256, Package_DIP:DIP-16_W7.62mm, F.Cu at (129.9, 95.0)
- added U29: 41256, Package_DIP:DIP-16_W7.62mm, F.Cu at (141.8, 94.9)
- added U3: 74LS74, Package_DIP:DIP-14_W7.62mm, F.Cu at (100.0, 29.8)
- added U30: 41256, Package_DIP:DIP-16_W7.62mm, F.Cu at (153.7, 94.9)
- added U31: 41256, Package_DIP:DIP-16_W7.62mm, F.Cu at (165.6, 94.9)
- added U32: 41256, Package_DIP:DIP-16_W7.62mm, F.Cu at (177.5, 94.9)
- added U33: 41256, Package_DIP:DIP-16_W7.62mm, F.Cu at (189.5, 94.9)
- added U34: 41256, Package_DIP:DIP-16_W7.62mm, F.Cu at (201.4, 94.9)
- added U35: 41256, Package_DIP:DIP-16_W7.62mm, F.Cu at (213.3, 94.9)
- added U36: 41256, Package_DIP:DIP-16_W7.62mm, F.Cu at (130.0, 126.9)
- added U37: 41256, Package_DIP:DIP-16_W7.62mm, F.Cu at (141.9, 126.8)
- added U38: 41256, Package_DIP:DIP-16_W7.62mm, F.Cu at (153.8, 126.8)
- added U39: 41256, Package_DIP:DIP-16_W7.62mm, F.Cu at (165.7, 126.8)
- added U4: 74LS08, Package_DIP:DIP-14_W7.62mm, F.Cu at (100.0, 44.0)
- added U40: 41256, Package_DIP:DIP-16_W7.62mm, F.Cu at (177.7, 126.8)
- added U41: 41256, Package_DIP:DIP-16_W7.62mm, F.Cu at (189.6, 126.8)
- added U42: 41256, Package_DIP:DIP-16_W7.62mm, F.Cu at (201.5, 126.8)
- added U43: 41256, Package_DIP:DIP-16_W7.62mm, F.Cu at (213.4, 126.8)
- added U44: 74LS157, Package_DIP:DIP-16_W7.62mm, F.Cu at (234.6, 28.5)
- added U45: 74LS139, Package_DIP:DIP-16_W7.62mm, F.Cu at (234.3, 46.3)
- added U46: 74LS157, Package_DIP:DIP-16_W7.62mm, F.Cu at (234.3, 70.8)
- added U47: 74LS153, Package_DIP:DIP-16_W7.62mm, F.Cu at (233.8, 147.9)
- added U5: 74LS02, Package_DIP:DIP-14_W7.62mm, F.Cu at (100.0, 56.1)
- added U6: 74LS393, Package_DIP:DIP-14_W7.62mm, F.Cu at (98.4, 82.5)
- added U7: 74153, Package_DIP:DIP-16_W7.62mm, F.Cu at (96.3, 96.0)
- added U8: 74153, Package_DIP:DIP-16_W7.62mm, F.Cu at (96.3, 109.4)
- added U9: 74153, Package_DIP:DIP-16_W7.62mm, F.Cu at (96.3, 122.9)
Other:
- board outline added: 237.1 x 147.2 mm

Commit message: Updated board layout with measurements
Add measurement for port spacing
Parts:
- moved U1 9.82 mm to (52.1, 44.8)
- moved J1 9.21 mm to (54.7, 51.1)
- moved C2 9.10 mm to (97.8, 34.3), turned to 270 degrees
- moved U44 8.39 mm to (234.3, 36.9)
- moved RN4 8.29 mm to (228.6, 29.2)
- moved C51 7.74 mm to (234.4, 41.1)
- moved U3 7.74 mm to (102.2, 37.2)
- moved C13 7.50 mm to (156.0, 30.7)
- moved C7 7.48 mm to (94.2, 101.8), turned to 270 degrees
- moved C17 7.47 mm to (203.8, 30.6)
- moved C18 7.38 mm to (215.6, 30.6)
- moved C15 7.36 mm to (179.9, 30.6)
- moved C12 7.33 mm to (144.1, 30.6)
- moved C11 7.33 mm to (132.2, 30.6)
- moved C5 7.30 mm to (94.3, 74.9), turned to 270 degrees
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Connections:
- J4 pad 1: (no net) -> Net-(J4-Pad1)
- J5 pad 10: SRW -> GND
- J5 pad 11: TODCLK -> ~BRAS
- J5 pad 12: BOOTCLK -> IRQ3
- J5 pad 13: S02 -> -12V
- J5 pad 14: S01 -> ~EXTRES
- J5 pad 15: BD3 -> 12V
- J5 pad 16: BD4 -> ~S.O.
- J5 pad 17: BD5 -> ~RES
- J5 pad 18: DB7 -> LPEN
- J5 pad 19: BA13 -> SRW
- J5 pad 20: BA14 -> ~EXTBUFCS
- J5 pad 21: BA1 -> TODCLK
- J5 pad 22: BA2 -> ~DISKROMCS
- J5 pad 23: BA3 -> BOOTCLK
- J5 pad 24: BA12 -> N.C.
- J5 pad 25: BA9 -> S02
- J5 pad 26: BA8 -> ~BCAS
- J5 pad 27: BP0 -> S01
- J5 pad 28: BP1 -> ~CS1
- J5 pad 29: ~NMI -> BD3
- J5 pad 3: GND -> 5V
- J5 pad 30: RDY -> ~EXTPRTCS
- J5 pad 31: ~IRQ -> BD4
- J5 pad 32: BP3 -> BD2
- J5 pad 33: BP2 -> BD5
- J5 pad 34: BA7 -> BD1
- J5 pad 35: BA6 -> BD6
- J5 pad 36: BA5 -> BD0
- J5 pad 37: BA4 -> BA13
- J5 pad 38: BA10 -> BD7
- J5 pad 39: BA11 -> BA14
- J5 pad 4: GND -> 5V
- J5 pad 40: BA0 -> BA15
- J5 pad 41: BA15 -> BA1
- J5 pad 42: BD7 -> BA0
- J5 pad 43: BD0 -> BA2
- J5 pad 44: BD1 -> BA11
- J5 pad 45: BD2 -> BA3
- J5 pad 46: ~EXTPRTCS -> BA10
- J5 pad 47: ~CS1 -> BA12
- J5 pad 48: ~BCAS -> BA4
- J5 pad 49: N.C. -> BA9
- J5 pad 50: ~DISKROMCS -> BA5
- J5 pad 51: ~EXTBUFCS -> BA8
- J5 pad 52: LPEN -> BA6
- J5 pad 53: ~S.O. -> BP0
- J5 pad 54: ~EXTRES -> BA7
- J5 pad 55: IRQ3 -> BP1
- J5 pad 56: GND -> BP2
- J5 pad 57: GND -> ~NMI
- J5 pad 58: GND -> BP3
- J5 pad 59: 5V -> RDY
- J5 pad 6: ~BRAS -> GND
- J5 pad 60: 5V -> ~IRQ
- J5 pad 7: -12V -> GND
- J5 pad 8: 12V -> GND
- J5 pad 9: ~RES -> GND
- J6 pad 10: SRW -> GND
- J6 pad 11: TODCLK -> ~BRAS
- J6 pad 12: BOOTCLK -> IRQ3
- J6 pad 13: S02 -> -12V
- J6 pad 14: S01 -> ~EXTRES
- J6 pad 15: BD3 -> 12V
- J6 pad 16: BD4 -> ~S.O.
- J6 pad 17: BD5 -> ~RES
- J6 pad 18: DB7 -> LPEN
- J6 pad 19: BA13 -> SRW
- J6 pad 20: BA14 -> ~EXTBUFCS
- J6 pad 21: BA1 -> TODCLK
- J6 pad 22: BA2 -> ~DISKROMCS
- J6 pad 23: BA3 -> BOOTCLK
- J6 pad 24: BA12 -> N.C.
- J6 pad 25: BA9 -> S02
- J6 pad 26: BA8 -> ~BCAS
- J6 pad 27: BP0 -> S01
- J6 pad 28: BP1 -> ~CS1
- J6 pad 29: ~NMI -> BD3
- J6 pad 3: GND -> 5V
- J6 pad 30: RDY -> ~EXTPRTCS
- J6 pad 31: ~IRQ -> BD4
- J6 pad 32: BP3 -> BD2
- J6 pad 33: BP2 -> BD5
- J6 pad 34: BA7 -> BD1
- J6 pad 35: BA6 -> BD6
- J6 pad 36: BA5 -> BD0
- J6 pad 37: BA4 -> BA13
- J6 pad 38: BA10 -> BD7
- J6 pad 39: BA11 -> BA14
- J6 pad 4: GND -> 5V
- J6 pad 40: BA0 -> BA15
- J6 pad 41: BA15 -> BA1
- J6 pad 42: BD7 -> BA0
- J6 pad 43: BD0 -> BA2
- J6 pad 44: BD1 -> BA11
- J6 pad 45: BD2 -> BA3
- J6 pad 46: ~EXTPRTCS -> BA10
- J6 pad 47: ~CS1 -> BA12
- J6 pad 48: ~BCAS -> BA4
- J6 pad 49: N.C. -> BA9
- J6 pad 50: ~DISKROMCS -> BA5
- J6 pad 51: ~EXTBUFCS -> BA8
- J6 pad 52: LPEN -> BA6
- J6 pad 53: ~S.O. -> BP0
- J6 pad 54: ~EXTRES -> BA7
- J6 pad 55: IRQ3 -> BP1
- J6 pad 56: GND -> BP2
- J6 pad 57: GND -> ~NMI
- J6 pad 58: GND -> BP3
- J6 pad 59: 5V -> RDY
- J6 pad 6: ~BRAS -> GND
- J6 pad 60: 5V -> ~IRQ
- J6 pad 7: -12V -> GND
- J6 pad 8: 12V -> GND
- J6 pad 9: ~RES -> GND
- J9 pad 10: GND -> DRAMO4
- J9 pad 11: GND -> EXTMA4
- J9 pad 12: GND -> DRAMO5
- J9 pad 13: GND -> EXTMA1
- J9 pad 14: GND -> DRAMO6
- J9 pad 15: GND -> EXTMA0
- J9 pad 16: GND -> DRAMO7
- J9 pad 17: N.C. -> GND
- J9 pad 18: ~PROCRES -> GND
- J9 pad 19: EXTBUF-RW -> GND
- J9 pad 2: EXTMA2 -> DRAMO0
- J9 pad 20: DRAM-RW -> GND
- J9 pad 21: ~ECAS -> GND
- J9 pad 22: ~ERAS -> ~BUSY1
- J9 pad 23: ~BUSY -> GND
- J9 pad 24: BP3 -> ~P2REFREQ
- J9 pad 25: BP2 -> GND
- J9 pad 26: BP1 -> ~P2REFGRNT
- J9 pad 27: BP0 -> GND
- J9 pad 28: ~P2REFGRNT -> BP0
- J9 pad 29: ~P2REFREQ -> GND
- J9 pad 3: EXTMA7 -> EXTMA2
- J9 pad 30: ~BUSY1 -> BP1
- J9 pad 32: GND -> BP2
- J9 pad 33: DRAMO7 -> N.C.
- J9 pad 34: DRAMO6 -> BP3
- J9 pad 35: DRAMO5 -> ~PROCRES
- J9 pad 36: DRAMO4 -> ~BUSY
- J9 pad 37: DRAMO3 -> EXTBUF-RW
- J9 pad 38: DRAMO2 -> ~ERAS
- J9 pad 39: DRAMO1 -> DRAM-RW
- J9 pad 4: EXTMA6 -> DRAMO1
- J9 pad 40: DRAMO0 -> ~ECAS
- J9 pad 5: EXTMA5 -> EXTMA7
- J9 pad 6: EXTMA4 -> DRAMO2
- J9 pad 7: EXTMA1 -> EXTMA6
- J9 pad 8: EXTMA0 -> DRAMO3
- J9 pad 9: GND -> EXTMA5
- P7 pad 10: SRW -> GND
- P7 pad 11: TODCLK -> ~BRAS
- P7 pad 12: BOOTCLK -> IRQ3
- P7 pad 13: S02 -> -12V
- P7 pad 14: S01 -> ~EXTRES
- P7 pad 15: BD3 -> 12V
- P7 pad 16: BD4 -> ~S.O.
- P7 pad 17: BD5 -> ~RES
- P7 pad 18: DB7 -> LPEN
- P7 pad 19: BA13 -> SRW
- P7 pad 20: BA14 -> ~EXTBUFCS
- P7 pad 21: BA1 -> TODCLK
- P7 pad 22: BA2 -> ~DISKROMCS
- P7 pad 23: BA3 -> BOOTCLK
- P7 pad 24: BA12 -> N.C.
- P7 pad 25: BA9 -> S02
- P7 pad 26: BA8 -> ~BCAS
- P7 pad 27: BP0 -> S01
- P7 pad 28: BP1 -> ~CS1
- P7 pad 29: ~NMI -> BD3
- P7 pad 3: GND -> 5V
- P7 pad 30: RDY -> ~EXTPRTCS
- P7 pad 31: ~IRQ -> BD4
- P7 pad 32: BP3 -> BD2
- P7 pad 33: BP2 -> BD5
- P7 pad 34: BA7 -> BD1
- P7 pad 35: BA6 -> BD6
- P7 pad 36: BA5 -> BD0
- P7 pad 37: BA4 -> BA13
- P7 pad 38: BA10 -> BD7
- P7 pad 39: BA11 -> BA14
- P7 pad 4: GND -> 5V
- P7 pad 40: BA0 -> BA15
- P7 pad 41: BA15 -> BA1
- P7 pad 42: BD7 -> BA0
- P7 pad 43: BD0 -> BA2
- P7 pad 44: BD1 -> BA11
- P7 pad 45: BD2 -> BA3
- P7 pad 46: ~EXTPRTCS -> BA10
- P7 pad 47: ~CS1 -> BA12
- P7 pad 48: ~BCAS -> BA4
- P7 pad 49: N.C. -> BA9
- P7 pad 50: ~DISKROMCS -> BA5
- P7 pad 51: ~EXTBUFCS -> BA8
- P7 pad 52: LPEN -> BA6
- P7 pad 53: ~S.O. -> BP0
- P7 pad 54: ~EXTRES -> BA7
- P7 pad 55: IRQ3 -> BP1
- P7 pad 56: GND -> BP2
- P7 pad 57: GND -> ~NMI
- P7 pad 58: GND -> BP3
- P7 pad 59: 5V -> RDY
- P7 pad 6: ~BRAS -> GND
- P7 pad 60: 5V -> ~IRQ
- P7 pad 7: -12V -> GND
- P7 pad 8: 12V -> GND
- P7 pad 9: ~RES -> GND
- P9 pad 10: GND -> DRAMO4
- P9 pad 11: GND -> EXTMA4
- P9 pad 12: GND -> DRAMO5
- P9 pad 13: GND -> EXTMA1
- P9 pad 14: GND -> DRAMO6
- P9 pad 15: GND -> EXTMA0
- P9 pad 16: GND -> DRAMO7
- P9 pad 17: N.C. -> GND
- P9 pad 18: ~PROCRES -> GND
- P9 pad 19: EXTBUF-RW -> GND
- P9 pad 2: EXTMA2 -> DRAMO0
- P9 pad 20: DRAM-RW -> GND
- P9 pad 21: ~ECAS -> GND
- P9 pad 22: ~ERAS -> ~BUSY1
- P9 pad 23: ~BUSY -> GND
- P9 pad 24: BP3 -> ~P2REFREQ
- P9 pad 25: BP2 -> GND
- P9 pad 26: BP1 -> ~P2REFGRNT
- P9 pad 27: BP0 -> GND
- P9 pad 28: ~P2REFGRNT -> BP0
- P9 pad 29: ~P2REFREQ -> GND
- P9 pad 3: EXTMA7 -> EXTMA2
- P9 pad 30: ~BUSY1 -> BP1
- P9 pad 32: GND -> BP2
- P9 pad 33: DRAMO7 -> N.C.
- P9 pad 34: DRAMO6 -> BP3
- P9 pad 35: DRAMO5 -> ~PROCRES
- P9 pad 36: DRAMO4 -> ~BUSY
- P9 pad 37: DRAMO3 -> EXTBUF-RW
- P9 pad 38: DRAMO2 -> ~ERAS
- P9 pad 39: DRAMO1 -> DRAM-RW
- P9 pad 4: EXTMA6 -> DRAMO1
- P9 pad 40: DRAMO0 -> ~ECAS
- P9 pad 5: EXTMA5 -> EXTMA7
- P9 pad 6: EXTMA4 -> DRAMO2
- P9 pad 7: EXTMA1 -> EXTMA6
- P9 pad 8: EXTMA0 -> DRAMO3
- P9 pad 9: GND -> EXTMA5
- RN9 pad 1: (no net) -> 5V
- U1 pad 1: (no net) -> 5V
- U1 pad 10: (no net) -> BA0
- U1 pad 11: (no net) -> BD0
- U1 pad 12: (no net) -> BD1
- U1 pad 13: (no net) -> BD2
- U1 pad 15: (no net) -> BD3
- U1 pad 16: (no net) -> BD4
- U1 pad 17: (no net) -> BD5
- U1 pad 18: (no net) -> BD6
- U1 pad 19: (no net) -> BD7
- U1 pad 2: (no net) -> BA12
- U1 pad 21: (no net) -> BA10
- U1 pad 23: (no net) -> BA11
- U1 pad 24: (no net) -> BA9
- U1 pad 25: (no net) -> BA8
- U1 pad 27: (no net) -> Net-(J4-Pad1)
- U1 pad 28: Vcc -> 5V
- U1 pad 3: (no net) -> BA7
- U1 pad 4: (no net) -> BA6
- U1 pad 5: (no net) -> BA5
- U1 pad 6: (no net) -> BA4
- U1 pad 7: (no net) -> BA3
- U1 pad 8: (no net) -> BA2
- U1 pad 9: (no net) -> BA1
- U10 pad 16: VCC -> 5V
- U11 pad 16: VCC -> 5V
- U12 pad 8: Vcc -> 5V
- U13 pad 8: Vcc -> 5V
- U14 pad 8: Vcc -> 5V
- U15 pad 8: Vcc -> 5V
- U16 pad 8: Vcc -> 5V
- U17 pad 8: Vcc -> 5V
- U18 pad 8: Vcc -> 5V
- U19 pad 8: Vcc -> 5V
- U2 pad 16: (no net) -> 5V
- U2 pad 8: (no net) -> GND
- U20 pad 8: Vcc -> 5V
- U21 pad 8: Vcc -> 5V
- U22 pad 8: Vcc -> 5V
- U23 pad 8: Vcc -> 5V
- U24 pad 8: Vcc -> 5V
- U25 pad 8: Vcc -> 5V
- U26 pad 8: Vcc -> 5V
- U27 pad 8: Vcc -> 5V
- U28 pad 8: Vcc -> 5V
- U29 pad 8: Vcc -> 5V
- U30 pad 8: Vcc -> 5V
- U31 pad 8: Vcc -> 5V
- U32 pad 8: Vcc -> 5V
- U33 pad 8: Vcc -> 5V
- U34 pad 8: Vcc -> 5V
- U35 pad 8: Vcc -> 5V
- U36 pad 8: Vcc -> 5V
- U37 pad 8: Vcc -> 5V
- U38 pad 8: Vcc -> 5V
- U39 pad 8: Vcc -> 5V
- U40 pad 8: Vcc -> 5V
- U41 pad 8: Vcc -> 5V
- U42 pad 8: Vcc -> 5V
- U43 pad 8: Vcc -> 5V
- U44 pad 16: (no net) -> 5V
- U44 pad 8: (no net) -> GND
- U46 pad 16: (no net) -> 5V
- U46 pad 8: (no net) -> GND
- U47 pad 16: (no net) -> 5V
- U47 pad 8: (no net) -> GND
- U7 pad 16: VCC -> 5V
- U8 pad 16: VCC -> 5V
- U9 pad 16: VCC -> 5V
Routing:
- net GND: track 0.00 -> 452.4 mm
- net 5V: track 0.00 -> 252.4 mm
Other:
- board size 237.1 x 147.2 mm -> 234 x 147.2 mm
- board text added: "WORK IN PROGRESS!!!!!!"
