File: kicad/B1024.sch (KiCad schematic (older format))
At the start: 109 parts, among them J5 EXP, J6 EXP, J9 COPRO, P7 EXP, P9 COPRO, U1 6264, U10 74153, U11 74153, U12 41256, U13 41256, U14 41256, U15 41256, U16 41256, U17 41256, U18 41256, U19 41256, U2 74LS85, U20 41256, U21 41256, U22 41256, U23 41256, U24 41256, U25 41256, U26 41256, U27 41256, U28 41256, U29 41256, U3 74LS74, U30 41256, U31 41256, U32 41256, U33 41256, U34 41256, U35 41256, U36 41256, U37 41256, U38 41256, U39 41256, U40 41256, U41 41256, U42 41256, U43 41256, U44 74LS157, U45 74LS139, U46 74LS157, U47 74LS153, U5 74LS02, U7 74153, U8 74153, U9 74153

Commit message: Add remaining parts, prelim board layout
Rotated pictures to match board layout. Added missing ics, resistors,
and jumpers. Preliminary layout. Updated readme.
Parts:
- added C52: 0.1uf, Capacitor_THT:C_Disc_D4.7mm_W2.5mm_P5.00mm, symbol Device:C_Small
- added J1: \"RESET\", Connector_PinHeader_2.54mm:PinHeader_1x02_P2.54mm_Horizontal, symbol Connector_Generic:Conn_01x02
- added J2: \"0FFF/0800 EN\", Connector_PinHeader_2.54mm:PinHeader_1x03_P2.54mm_Horizontal, symbol Connector_Generic:Conn_01x03
- added J3: \"LED\", Connector_PinHeader_2.54mm:PinHeader_1x03_P2.54mm_Horizontal, symbol Connector_Generic:Conn_01x03
- added J4: \"RAM ROM\", Connector_PinHeader_2.54mm:PinHeader_1x03_P2.54mm_Horizontal, symbol Connector_Generic:Conn_01x03
- added R1, R4: 22ohm, Resistor_THT:R_Axial_DIN0207_L6.3mm_D2.5mm_P10.16mm_Horizontal, symbol Device:R
- added R2, R3: 4K7, Resistor_THT:R_Axial_DIN0207_L6.3mm_D2.5mm_P10.16mm_Horizontal, symbol Device:R
- added RN1: 4K7, Resistor_THT:R_Array_SIP10, symbol Device:R_Network09_US
- added RN2, RN3: 22 ohm, Resistor_THT:R_Array_SIP10, symbol Device:R_Pack05_SIP
- added RN4, RN5: 22 ohm, Resistor_THT:R_Array_SIP8, symbol Device:R_Pack04_SIP
- added RN6, RN9: 4K7, Resistor_THT:R_Array_SIP8, symbol Device:R_Network07_US
- added RN7, RN8: 10K, Resistor_THT:R_Array_SIP10, symbol Device:R_Network09_US
- C1, C10, C11, C12, C13, C14, C15, C16, C17, C18, C19, C2, C20, C21, C22, C23, C24, C25, C26, C27, C28, C29, C3, C30, C31, C32, C33, C34, C35, C36, C37, C38, C39, C4, C40, C41, C42, C43, C44, C45, C46, C47, C48, C49, C5, C50, C51, C6, C7, C8, C9: footprint (none) -> Capacitor_THT:C_Disc_D4.7mm_W2.5mm_P5.00mm
- J5, J6, P7: footprint (none) -> Connector_PinHeader_2.54mm:PinHeader_2x30_P2.54mm_Vertical
- J9, P9: footprint (none) -> Connector_PinHeader_2.54mm:PinHeader_2x20_P2.54mm_Vertical
- U1: footprint (none) -> Package_DIP:DIP-28_W15.24mm
- U10, U11, U12, U13, U14, U15, U16, U17, U18, U19, U2, U20, U21, U22, U23, U24, U25, U26, U27, U28, U29, U30, U31, U32, U33, U34, U35, U36, U37, U38, U39, U40, U41, U42, U43, U44, U45, U46, U47, U7, U8, U9: footprint (none) -> Package_DIP:DIP-16_W7.62mm
- U3, U5: footprint (none) -> Package_DIP:DIP-14_W7.62mm
- U4, U6: renamed from U?; footprint (none) -> Package_DIP:DIP-14_W7.62mm
Connections:
- net 5V is gone; now on net +5V: C1.1, C10.1, C11.1, C12.1, C13.1, C14.1, C15.1, C16.1, C17.1, C18.1, C19.1, C2.1, C20.1, C21.1, C22.1, C23.1, C24.1, C25.1, C26.1, C27.1, C28.1, C29.1, C3.1, C30.1, C31.1, C32.1, C33.1, C34.1, C35.1, C36.1, C37.1, C38.1, C39.1, C4.1, C40.1, C41.1, C42.1, C43.1, C44.1, C45.1, C46.1, C47.1, C48.1, C49.1, C5.1, C50.1, C51.1, C6.1, C7.1, C8.1, C9.1, J5.1 (Pin_1), J5.2 (Pin_2), J5.59 (Pin_59), J5.60 (Pin_60), J6.1 (Pin_1), J6.2 (Pin_2), J6.59 (Pin_59), J6.60 (Pin_60), P7.1 (Pin_1), P7.2 (Pin_2), P7.59 (Pin_59), P7.60 (Pin_60)
- net GND: now also U3.7 (GND), U4.7 (GND), U45.16 (VCC), U5.7 (GND), U6.7 (GND), C52.2
- net +5V: now reaches U45.8 (GND)
- net +5V: now also U3.14 (VCC), U4.14 (VCC), U5.14 (VCC), U6.14 (VCC), C52.1
Other:
- moved on the sheet: U3C, U45C, U4A, U4B, U4C, U4D, U4E, U5A, U5B, U5C, U5D, U6A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

Commit message: Updated board layout with measurements
Add measurement for port spacing
Parts:
- removed J5, J6, P7: EXP, Connector_PinHeader_2.54mm:PinHeader_2x30_P2.54mm_Vertical, symbol Connector_Generic:Conn_02x30_Counter_Clockwise
- removed J9, P9: COPRO, Connector_PinHeader_2.54mm:PinHeader_2x20_P2.54mm_Vertical, symbol Connector_Generic:Conn_02x20_Counter_Clockwise
- added J5, J6, P7: EXP, Connector_PinHeader_2.54mm:PinHeader_2x30_P2.54mm_Vertical, symbol Connector_Generic:Conn_02x30_Odd_Even
- added J9, P9: COPRO, Connector_PinHeader_2.54mm:PinHeader_2x20_P2.54mm_Vertical, symbol Connector_Generic:Conn_02x20_Odd_Even
Connections:
- net VCC is gone; now on net +5V: U10.16 (VCC), U11.16 (VCC), U7.16 (VCC), U8.16 (VCC), U9.16 (VCC)
- net Vcc is gone; now on net +5V: U1.28 (Vcc), U12.8 (Vcc), U13.8 (Vcc), U14.8 (Vcc), U15.8 (Vcc), U16.8 (Vcc), U17.8 (Vcc), U18.8 (Vcc), U19.8 (Vcc), U20.8 (Vcc), U21.8 (Vcc), U22.8 (Vcc), U23.8 (Vcc), U24.8 (Vcc), U25.8 (Vcc), U26.8 (Vcc), U27.8 (Vcc), U28.8 (Vcc), U29.8 (Vcc), U30.8 (Vcc), U31.8 (Vcc), U32.8 (Vcc), U33.8 (Vcc), U34.8 (Vcc), U35.8 (Vcc), U36.8 (Vcc), U37.8 (Vcc), U38.8 (Vcc), U39.8 (Vcc), U40.8 (Vcc), U41.8 (Vcc), U42.8 (Vcc), U43.8 (Vcc)
- net +5V: now also RN9.1 (common), U1.1 (NC), U2.16 (VCC), U44.16 (VCC), U46.16 (VCC), U47.16 (VCC), J5.1 (Pin_1), J5.2 (Pin_2), J5.3 (Pin_3), J5.4 (Pin_4), J6.1 (Pin_1), J6.2 (Pin_2), J6.3 (Pin_3), J6.4 (Pin_4), P7.1 (Pin_1), P7.2 (Pin_2), P7.3 (Pin_3), P7.4 (Pin_4)
- net -12V: now also J5.13 (Pin_13), J6.13 (Pin_13), P7.13 (Pin_13)
- net 12V: now also J5.15 (Pin_15), J6.15 (Pin_15), P7.15 (Pin_15)
- net BA0: now also U1.10 (A0), J5.42 (Pin_42), J6.42 (Pin_42), P7.42 (Pin_42)
- net BA1: now also U1.9 (A1), J5.41 (Pin_41), J6.41 (Pin_41), P7.41 (Pin_41)
- net BA10: now also U1.21 (A10), J5.46 (Pin_46), J6.46 (Pin_46), P7.46 (Pin_46)
- net BA11: now also U1.23 (A11), J5.44 (Pin_44), J6.44 (Pin_44), P7.44 (Pin_44)
- net BA12: now also U1.2 (A12), J5.47 (Pin_47), J6.47 (Pin_47), P7.47 (Pin_47)
- net BA13: now also J5.37 (Pin_37), J6.37 (Pin_37), P7.37 (Pin_37)
- net BA14: now also J5.39 (Pin_39), J6.39 (Pin_39), P7.39 (Pin_39)
- net BA15: now also J5.40 (Pin_40), J6.40 (Pin_40), P7.40 (Pin_40)
- net BA2: now also U1.8 (A2), J5.43 (Pin_43), J6.43 (Pin_43), P7.43 (Pin_43)
- net BA3: now also U1.7 (A3), J5.45 (Pin_45), J6.45 (Pin_45), P7.45 (Pin_45)
- net BA4: now also U1.6 (A4), J5.48 (Pin_48), J6.48 (Pin_48), P7.48 (Pin_48)
- net BA5: now also U1.5 (A5), J5.50 (Pin_50), J6.50 (Pin_50), P7.50 (Pin_50)
- net BA6: now also U1.4 (A6), J5.52 (Pin_52), J6.52 (Pin_52), P7.52 (Pin_52)
- net BA7: now also U1.3 (A7), J5.54 (Pin_54), J6.54 (Pin_54), P7.54 (Pin_54)
- net BA8: now also U1.25 (A8), J5.51 (Pin_51), J6.51 (Pin_51), P7.51 (Pin_51)
- net BA9: now also U1.24 (A9), J5.49 (Pin_49), J6.49 (Pin_49), P7.49 (Pin_49)
- net BD0: now also U1.11 (D0), J5.36 (Pin_36), J6.36 (Pin_36), P7.36 (Pin_36)
- net BD1: now also U1.12 (D1), J5.34 (Pin_34), J6.34 (Pin_34), P7.34 (Pin_34)
- net BD2: now also U1.13 (D2), J5.32 (Pin_32), J6.32 (Pin_32), P7.32 (Pin_32)
- net BD3: now also U1.15 (D3), J5.29 (Pin_29), J6.29 (Pin_29), P7.29 (Pin_29)
- net BD4: now also U1.16 (D4), J5.31 (Pin_31), J6.31 (Pin_31), P7.31 (Pin_31)
- net BD5: now also U1.17 (D5), J5.33 (Pin_33), J6.33 (Pin_33), P7.33 (Pin_33)
- net BD7: now also U1.19 (D7), J5.38 (Pin_38), J6.38 (Pin_38), P7.38 (Pin_38)
- net BOOTCLK: now also J5.23 (Pin_23), J6.23 (Pin_23), P7.23 (Pin_23)
- net BP0: now also J5.53 (Pin_53), J6.53 (Pin_53), J9.28 (Pin_28), P7.53 (Pin_53), P9.28 (Pin_28)
- net BP1: now also J5.55 (Pin_55), J6.55 (Pin_55), J9.30 (Pin_30), P7.55 (Pin_55), P9.30 (Pin_30)
- net BP2: now also J5.56 (Pin_56), J6.56 (Pin_56), J9.32 (Pin_32), P7.56 (Pin_56), P9.32 (Pin_32)
- net BP3: now also J5.58 (Pin_58), J6.58 (Pin_58), J9.34 (Pin_34), P7.58 (Pin_58), P9.34 (Pin_34)
- net DRAM-RW: now also J9.39 (Pin_39), P9.39 (Pin_39)
- net DRAMO0: now also J9.2 (Pin_2), P9.2 (Pin_2)
- net DRAMO1: now also J9.4 (Pin_4), P9.4 (Pin_4)
- net DRAMO2: now also J9.6 (Pin_6), P9.6 (Pin_6)
- net DRAMO3: now also J9.8 (Pin_8), P9.8 (Pin_8)
- net DRAMO4: now also J9.10 (Pin_10), P9.10 (Pin_10)
- net DRAMO5: now also J9.12 (Pin_12), P9.12 (Pin_12)
- net DRAMO6: now also J9.14 (Pin_14), P9.14 (Pin_14)
- net DRAMO7: now also J9.16 (Pin_16), P9.16 (Pin_16)
- net EXTBUF-RW: now also J9.37 (Pin_37), P9.37 (Pin_37)
- net EXTMA: now also J9.1 (Pin_1), P9.1 (Pin_1)
- net EXTMA0: now also J9.15 (Pin_15), P9.15 (Pin_15)
- net EXTMA1: now also J9.13 (Pin_13), P9.13 (Pin_13)
- net EXTMA2: now also J9.3 (Pin_3), P9.3 (Pin_3)
- net EXTMA4: now also J9.11 (Pin_11), P9.11 (Pin_11)
- net EXTMA5: now also J9.9 (Pin_9), P9.9 (Pin_9)
- net EXTMA6: now also J9.7 (Pin_7), P9.7 (Pin_7)
- net EXTMA7: now also J9.5 (Pin_5), P9.5 (Pin_5)
- net GND: now also U2.8 (GND), U44.8 (GND), U46.8 (GND), U47.8 (GND), J5.10 (Pin_10), J5.5 (Pin_5), J5.6 (Pin_6), J5.7 (Pin_7), J5.8 (Pin_8), J5.9 (Pin_9), J6.10 (Pin_10), J6.5 (Pin_5), J6.6 (Pin_6), J6.7 (Pin_7), J6.8 (Pin_8), J6.9 (Pin_9), J9.17 (Pin_17), J9.18 (Pin_18), J9.19 (Pin_19), J9.20 (Pin_20), J9.21 (Pin_21), J9.23 (Pin_23), J9.25 (Pin_25), J9.27 (Pin_27), J9.29 (Pin_29), J9.31 (Pin_31), P7.10 (Pin_10), P7.5 (Pin_5), P7.6 (Pin_6), P7.7 (Pin_7), P7.8 (Pin_8), P7.9 (Pin_9), P9.17 (Pin_17), P9.18 (Pin_18), P9.19 (Pin_19), P9.20 (Pin_20), P9.21 (Pin_21), P9.23 (Pin_23), P9.25 (Pin_25), P9.27 (Pin_27), P9.29 (Pin_29), P9.31 (Pin_31)
- net IRQ3: now also J5.12 (Pin_12), J6.12 (Pin_12), P7.12 (Pin_12)
- net LPEN: now also J5.18 (Pin_18), J6.18 (Pin_18), P7.18 (Pin_18)
- net N.C.: now also J5.24 (Pin_24), J6.24 (Pin_24), J9.33 (Pin_33), P7.24 (Pin_24), P9.33 (Pin_33)
- net RDY: now also J5.59 (Pin_59), J6.59 (Pin_59), P7.59 (Pin_59)
- net S01: now also J5.27 (Pin_27), J6.27 (Pin_27), P7.27 (Pin_27)
- net S02: now also J5.25 (Pin_25), J6.25 (Pin_25), P7.25 (Pin_25)
- net SRW: now also J5.19 (Pin_19), J6.19 (Pin_19), P7.19 (Pin_19)
- net TODCLK: now also J5.21 (Pin_21), J6.21 (Pin_21), P7.21 (Pin_21)
- net ~BCAS: now also J5.26 (Pin_26), J6.26 (Pin_26), P7.26 (Pin_26)
- net ~BRAS: now also J5.11 (Pin_11), J6.11 (Pin_11), P7.11 (Pin_11)
- net ~BUSY: now also J9.36 (Pin_36), P9.36 (Pin_36)
- net ~BUSY1: now also J9.22 (Pin_22), P9.22 (Pin_22)
- net ~CS1: now also J5.28 (Pin_28), J6.28 (Pin_28), P7.28 (Pin_28)
- net ~DISKROMCS: now also J5.22 (Pin_22), J6.22 (Pin_22), P7.22 (Pin_22)
- net ~ECAS: now also J9.40 (Pin_40), P9.40 (Pin_40)
- net ~ERAS: now also J9.38 (Pin_38), P9.38 (Pin_38)
- net ~EXTBUFCS: now also J5.20 (Pin_20), J6.20 (Pin_20), P7.20 (Pin_20)
- net ~EXTPRTCS: now also J5.30 (Pin_30), J6.30 (Pin_30), P7.30 (Pin_30)
- net ~EXTRES: now also J5.14 (Pin_14), J6.14 (Pin_14), P7.14 (Pin_14)
- net ~IRQ: now also J5.60 (Pin_60), J6.60 (Pin_60), P7.60 (Pin_60)
- net ~NMI: now also J5.57 (Pin_57), J6.57 (Pin_57), P7.57 (Pin_57)
- net ~P2REFGRNT: now also J9.26 (Pin_26), P9.26 (Pin_26)
- net ~P2REFREQ: now also J9.24 (Pin_24), P9.24 (Pin_24)
- net ~PROCRES: now also J9.35 (Pin_35), P9.35 (Pin_35)
- net ~RES: now also J5.17 (Pin_17), J6.17 (Pin_17), P7.17 (Pin_17)
- net ~S.O.: now also J5.16 (Pin_16), J6.16 (Pin_16), P7.16 (Pin_16)
- net BD6: now reaches U1.18 (D6)
- net BD6: now also J5.35 (Pin_35), J6.35 (Pin_35), P7.35 (Pin_35)
- net at U1.27 (R/~W): now also J4.1 (Pin_1)
Other:
- note added: "IGNORE the PIN#'s! Only the position is important."
- moved on the sheet: J4, U1, U10, U11, U2, U44, U45A, U45B, U46, U47, U7, U8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

Commit message: Routing and circuit updates
Schematic is starting to take shape. Route most common dram line and
many expansion lines.
Parts:
- added TP1: TestPoint, Connector_PinHeader_2.54mm:PinHeader_1x01_P2.54mm_Vertical, symbol Connector:TestPoint
Connections:
- net labels added: ROUTE
- net labels removed: D
- wire segments 253 -> 365
Other:
- moved on the sheet: C4, J3, J4, R1, R2, R3, R4, RN1, RN2, RN3, RN4, RN5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
